File: RGB_Matrix.kicad_sch (KiCad schematic)
At the start: 95 parts

Commit message: Change
Parts:
- removed D1, D10, D11, D12, D13, D14, D15, D16, D17, D18, D19, D2, D20, D21, D22, D23, D24, D25, D26, D27, D28, D29, D3, D30, D31, D32, D33, D34, D35, D39, D4, D40, D41, D42, D43, D44, D45, D46, D47, D48, D49, D5, D50, D51, D52, D53, D54, D55, D56, D57, D58, D59, D6, D60, D61, D62, D63, D64, D65, D66, D67, D68, D7, D8, D9: LED_ABGR, horrortroll_lib:LED_1206R, symbol Device:LED_ABGR
- removed R10, R102, R108, R109, R11, R36, R41, R42, R48, R53, R54, R59, R60, R65, R66, R71, R72, R77, R78, R8, R83, R84, R88, R89, R9, R90, R93, R96, R98, R99: R, Common_Footprint:R_0402, symbol Device:R
