File: MUX.kicad_sch (KiCad schematic)
At the start: 18 parts, among them U2 74HC4051, U32 74HC4051, U38 74HC4051, U45 74HC4051, U51 74HC4051, U56 74HC4051, U62 74HC4051, U69 74HC4051, U74 74HC4051

Commit message: Make it 60%
Parts:
- removed U74: 74HC4051, Package_SO:SSOP-16_4.4x5.2mm_P0.65mm, symbol 74xx:74HC4051
Connections:
- net +3V3: no longer C17.2
- net 413: now also U69.13 (A0); no longer U69.14 (A1)
- net 414: now also U69.14 (A1); no longer U69.13 (A0)
- net GND: now also C17.2; no longer C17.1
Other:
- moved on the sheet: C17

Commit message: fi
Parts:
- removed C17: 0.1uF, Common_Footprint:C_0402, symbol Device:C_Small
Other:
- moved on the sheet: C17
Changed lines of the file:
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@@
 	)
 	(junction
+		(at 99.06 137.795)
+		(diameter 0)
+		(color 0 0 0 0)
+	)
+	(junction
 		(at 210.82 55.88)
 		(diameter 0)
@@
 	)
 	(junction
+		(at 99.06 132.715)
+		(diameter 0)
+		(color 0 0 0 0)
+	)
+	(junction
 		(at 113.03 55.88)
 		(diameter 0)
@@
 	)
 	(junction
-		(at 78.74 137.795)
+		(at 88.9 132.715)
 		(diameter 0)
 		(color 0 0 0 0)
@@
 	)
 	(junction
-		(at 99.06 132.715)
-		(diameter 0)
-		(color 0 0 0 0)
-	)
-	(junction
-		(at 99.06 137.795)
-		(diameter 0)
-		(color 0 0 0 0)
-	)
-	(junction
 		(at 35.56 55.88)
 		(diameter 0)
@@
 	)
 	(junction
-		(at 88.9 137.795)
-		(diameter 0)
-		(color 0 0 0 0)
-	)
-	(junction
 		(at 152.4 55.88)
 		(diameter 0)
@@
 	)
 	(junction
-		(at 78.74 132.715)
+		(at 88.9 137.795)
 		(diameter 0)
 		(color 0 0 0 0)
@@
 	(wire
 		(pts
-			(xy 68.58 137.795) (xy 78.74 137.795)
+			(xy 78.74 137.795) (xy 88.9 137.795)
 		)
 		(stroke
@@
 	(wire
 		(pts
-			(xy 68.58 132.715) (xy 78.74 132.715)
+			(xy 78.74 132.715) (xy 88.9 132.715)
 		)
 		(stroke
@@
 	(wire
 		(pts
+			(xy 88.9 132.715) (xy 99.06 132.715)
+		)
+		(stroke
+			(width 0)
+			(type default)
+		)
+	)
+	(wire
+		(pts
 			(xy 181.61 55.88) (xy 200.66 55.88)
 		)
@@
 	(wire
 		(pts
-			(xy 88.9 137.795) (xy 99.06 137.795)
-		)
-		(stroke
-			(width 0)
-			(type default)
-		)
-	)
-	(wire
-		(pts
 			(xy 99.06 132.715) (xy 109.22 132.715)
 		)
@@
 	(wire
 		(pts
-			(xy 78.74 132.715) (xy 99.06 132.715)
-		)
-		(stroke
-			(width 0)
-			(type default)
-		)
-	)
-	(wire
-		(pts
-			(xy 78.74 137.795) (xy 88.9 137.795)
+			(xy 88.9 137.795) (xy 99.06 137.795)
 		)
 		(stroke
@@
 	(symbol
 		(lib_id "power:GND")
-		(at 68.58 137.795 270)
+		(at 78.74 137.795 270)
 		(unit 1)
 		(exclude_from_sim no)
@@
 		(dnp no)
 		(property "Reference" "#PWR0278"
-			(at 62.23 137.795 0)
+			(at 72.39 137.795 0)
 			(effects
 				(font
@@
 		)
 		(property "Value" "GND"
-			(at 62.23 137.795 90)
+			(at 72.39 137.795 90)
 			(effects
 				(font
@@
 		)
 		(property "Footprint" ""
-			(at 68.58 137.795 0)
+			(at 78.74 137.795 0)
 			(effects
 				(font
@@
 		)
 		(property "Datasheet" ""
-			(at 68.58 137.795 0)
+			(at 78.74 137.795 0)
 			(effects
 				(font
@@
 		)
 		(property "Description" ""
-			(at 68.58 137.795 0)
+			(at 78.74 137.795 0)
 			(effects
 				(font
@@
 	(symbol
 		(lib_id "Device:C_Small")
-		(at 88.9 140.335 180)
-		(unit 1)
-		(exclude_from_sim no)
-		(in_bom yes)
-		(on_board yes)
-		(dnp no)
-		(property "Reference" "C17"
-			(at 86.36 141.5988 0)
-			(effects
-				(font
-					(size 1.27 1.27)
-				)
-				(justify left)
-			)
-		)
-		(property "Value" "0.1uF"
-			(at 86.36 139.0588 0)
-			(effects
-				(font
-					(size 1.27 1.27)
-				)
-				(justify left)
-			)
-		)
-		(property "Footprint" "Common_Footprint:C_0402"
-			(at 88.9 140.335 0)
-			(effects
-				(font
-					(size 1.27 1.27)
-				)
-				(hide yes)
-			)
-		)
-		(property "Datasheet" "~"
-			(at 88.9 140.335 0)
-			(effects
-				(font
-					(size 1.27 1.27)
-				)
-				(hide yes)
-			)
-		)
-		(property "Description" ""
-			(at 88.9 140.335 0)
-			(effects
-				(font
-					(size 1.27 1.27)
-				)
-				(hide yes)
-			)
-		)
-		(pin "1"
-		)
-		(pin "2"
-		)
-		(instances
-			(project "Matrix"
-				(path "/24243bf5-bf8b-4a70-84ec-02c831689d67"
-					(reference "C17")
-					(unit 1)
-				)
-			)
-			(project "Heart HE 65"
-				(path "/4ead6829-f799-4396-8251-4a39c9105839/9fdba786-3862-4d85-a21d-909462cdc5e8"
-					(reference "C3")
-					(unit 1)
-				)
-			)
-			(project "Salane usO"
-				(path "/508e0333-ab34-4ef1-bc47-aa6189986b3c"
-					(reference "C19")
-					(unit 1)
-				)
-			)
-		)
-	)
-	(symbol
-		(lib_id "Device:C_Small")
 		(at 139.7 135.255 180)
 		(unit 1)
@@
 	(symbol
 		(lib_id "power:+3V3")
-		(at 68.58 132.715 90)
+		(at 78.74 132.715 90)
 		(unit 1)
 		(exclude_from_sim no)
@@
 		(dnp no)
 		(property "Reference" "#PWR0279"
-			(at 72.39 132.715 0)
+			(at 82.55 132.715 0)
 			(effects
 				(font
@@
 		)
 		(property "Value" "+3V3"
-			(at 62.23 132.715 90)
+			(at 72.39 132.715 90)
 			(effects
 				(font
@@
 		)
 		(property "Footprint" ""
-			(at 68.58 132.715 0)
+			(at 78.74 132.715 0)
 			(effects
 				(font
@@
 		)
 		(property "Datasheet" ""
-			(at 68.58 132.715 0)
+			(at 78.74 132.715 0)
 			(effects
 				(font
@@
 		)
 		(property "Description" ""
-			(at 68.58 132.715 0)
+			(at 78.74 132.715 0)
 			(effects
 				(font
@@
 	(symbol
 		(lib_id "Device:C_Small")
-		(at 78.74 135.255 180)
+		(at 88.9 135.255 180)
 		(unit 1)
 		(exclude_from_sim no)
@@
 		(dnp no)
 		(property "Reference" "C17"
-			(at 76.2 136.5188 0)
+			(at 86.36 136.5188 0)
 			(effects
 				(font
@@
 		)
 		(property "Value" "0.1uF"
-			(at 76.2 133.9788 0)
+			(at 86.36 133.9788 0)
 			(effects
 				(font
@@
 		)
 		(property "Footprint" "Common_Footprint:C_0402"
-			(at 78.74 135.255 0)
+			(at 88.9 135.255 0)
 			(effects
 				(font
@@
 		)
 		(property "Datasheet" "~"
-			(at 78.74 135.255 0)
+			(at 88.9 135.255 0)
 			(effects
 				(font
@@
 		)
 		(property "Description" ""
-			(at 78.74 135.255 0)
+			(at 88.9 135.255 0)
 			(effects
 				(font
